File: radio-9014x1-ss-rounded2.kicad_sch (KiCad schematic)
At the start: 17 parts, among them J1 AudioJack2, Q1 BC547/S9014

Commit message: Easier soldering
Edited transistor footprint to the 'wide' variety for easier soldering
Parts:
- Q1: footprint Package_TO_SOT_THT:TO-92_Inline -> Package_TO_SOT_THT:TO-92_Inline_Wide
Changed lines of the file:
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@@
     (pin "1")
     (instances
-      (project "radio-9014x1"
+      (project "radio-9014x1-ss-wide-transistir"
         (path "/b6366648-9fec-4168-91d1-0e8832484c0a"
           (reference "#FLG01") (unit 1)
@@
     (pin "R")
     (instances
-      (project "radio-9014x1"
+      (project "radio-9014x1-ss-wide-transistir"
         (path "/b6366648-9fec-4168-91d1-0e8832484c0a"
           (reference "J1") (unit 1)
@@
     (pin "1")
     (instances
-      (project "radio-9014x1"
+      (project "radio-9014x1-ss-wide-transistir"
         (path "/b6366648-9fec-4168-91d1-0e8832484c0a"
           (reference "C5") (unit 1)
@@
     (pin "2")
     (instances
-      (project "radio-9014x1"
+      (project "radio-9014x1-ss-wide-transistir"
         (path "/b6366648-9fec-4168-91d1-0e8832484c0a"
           (reference "D1") (unit 1)
@@
     (pin "2")
     (instances
-      (project "radio-9014x1"
+      (project "radio-9014x1-ss-wide-transistir"
         (path "/b6366648-9fec-4168-91d1-0e8832484c0a"
           (reference "L2") (unit 1)
@@
     (pin "1")
     (instances
-      (project "radio-9014x1"
+      (project "radio-9014x1-ss-wide-transistir"
         (path "/b6366648-9fec-4168-91d1-0e8832484c0a"
           (reference "#PWR02") (unit 1)
@@
     (pin "1")
     (instances
-      (project "radio-9014x1"
+      (project "radio-9014x1-ss-wide-transistir"
         (path "/b6366648-9fec-4168-91d1-0e8832484c0a"
           (reference "C2") (unit 1)
@@
     (pin "2")
     (instances
-      (project "radio-9014x1"
+      (project "radio-9014x1-ss-wide-transistir"
         (path "/b6366648-9fec-4168-91d1-0e8832484c0a"
           (reference "R2") (unit 1)
@@
     (pin "1")
     (instances
-      (project "radio-9014x1"
+      (project "radio-9014x1-ss-wide-transistir"
         (path "/b6366648-9fec-4168-91d1-0e8832484c0a"
           (reference "#PWR01") (unit 1)
@@
     (pin "1")
     (instances
-      (project "radio-9014x1"
+      (project "radio-9014x1-ss-wide-transistir"
         (path "/b6366648-9fec-4168-91d1-0e8832484c0a"
           (reference "C4") (unit 1)
@@
     (pin "3")
     (instances
-      (project "radio-9014x1"
+      (project "radio-9014x1-ss-wide-transistir"
         (path "/b6366648-9fec-4168-91d1-0e8832484c0a"
           (reference "L1") (unit 1)
@@
     (pin "2")
     (instances
-      (project "radio-9014x1"
+      (project "radio-9014x1-ss-wide-transistir"
         (path "/b6366648-9fec-4168-91d1-0e8832484c0a"
           (reference "Battery1") (unit 1)
@@
     (pin "2")
     (instances
-      (project "radio-9014x1"
+      (project "radio-9014x1-ss-wide-transistir"
         (path "/b6366648-9fec-4168-91d1-0e8832484c0a"
           (reference "R1") (unit 1)
@@
     (pin "2")
     (instances
-      (project "radio-9014x1"
+      (project "radio-9014x1-ss-wide-transistir"
         (path "/b6366648-9fec-4168-91d1-0e8832484c0a"
           (reference "RV1") (unit 1)
@@
     (pin "3")
     (instances
-      (project "radio-9014x1"
+      (project "radio-9014x1-ss-wide-transistir"
         (path "/b6366648-9fec-4168-91d1-0e8832484c0a"
           (reference "C1") (unit 1)
@@
       (effects (font (size 1.27 1.27)) (justify left))
     )
-    (property "Footprint" "Package_TO_SOT_THT:TO-92_Inline" (at 143.51 83.82 0)
+    (property "Footprint" "Package_TO_SOT_THT:TO-92_Inline_Wide" (at 143.51 83.82 0)
       (effects (font (size 1.27 1.27) italic) (justify left) hide)
     )
@@
     (pin "1")
     (instances
-      (project "radio-9014x1"
+      (project "radio-9014x1-ss-wide-transistir"
         (path "/b6366648-9fec-4168-91d1-0e8832484c0a"
           (reference "Q1") (unit 1)
@@
     (pin "1")
     (instances
-      (project "radio-9014x1"
+      (project "radio-9014x1-ss-wide-transistir"
         (path "/b6366648-9fec-4168-91d1-0e8832484c0a"
           (reference "#PWR03") (unit 1)
@@
     (pin "2")
     (instances
-      (project "radio-9014x1"
+      (project "radio-9014x1-ss-wide-transistir"
         (path "/b6366648-9fec-4168-91d1-0e8832484c0a"
           (reference "Switch1") (unit 1)
@@
     (pin "1")
     (instances
-      (project "radio-9014x1"
+      (project "radio-9014x1-ss-wide-transistir"
         (path "/b6366648-9fec-4168-91d1-0e8832484c0a"
           (reference "C3") (unit 1)
@@
     (pin "1")
     (instances
-      (project "radio-9014x1"
+      (project "radio-9014x1-ss-wide-transistir"
         (path "/b6366648-9fec-4168-91d1-0e8832484c0a"
           (reference "#PWR04") (unit 1)
@@
     (pin "1")
     (instances
-      (project "radio-9014x1"
+      (project "radio-9014x1-ss-wide-transistir"
         (path "/b6366648-9fec-4168-91d1-0e8832484c0a"
           (reference "C6") (unit 1)
@@
     (pin "2")
     (instances
-      (project "radio-9014x1"
+      (project "radio-9014x1-ss-wide-transistir"
         (path "/b6366648-9fec-4168-91d1-0e8832484c0a"
           (reference "D2") (unit 1)
